File: IIsiSEthernet.kicad_pcb (KiCad board)
At the start: 4 copper layers, 124 x 38 mm, 53 parts, among them IC1 SST39SF010A-70-4C-WHE, J1 650906-5, J3 USB_B_Micro, J5 RJ45_Amphenol_RJMG1BD3B8K1ANR, J7 AVR-JTAG-10, U2 ATF1502ASL-25AU44, U3 ENC624J600-I_PT, U4 LD1117S33TR_SOT223, X2 ASE-xxxMHz

Commit message: minor stuff
Routing:
- net GND: track 95.2 -> 100.4 mm, vias 56 -> 58

Commit message: cleanups, switch for ROM bank
Parts:
- added R4: 10k, Resistor_SMD:R_0402_1005Metric, F.Cu at (198.2, 138.2)
- added R5: 10k, Resistor_SMD:R_0402_1005Metric, F.Cu at (207.8, 138.2)
- added S3: SSAJ110100, For_SeeedStudio:SW_SSAJ110100, F.Cu at (203.0, 139.0)
- moved C5 0.96 mm to (141.3, 135.8), turned to 180 degrees
Connections:
- IC1 pad 10: GND -> ROM_BANK
Routing:
- net ROM_BANK: track 0.00 -> 66.7 mm, vias 0 -> 2
- net Net-(R5-Pad1): track 0.00 -> 3.75 mm
- net Net-(R4-Pad1): track 0.00 -> 3.75 mm
- net GND: track 100.4 -> 102.3 mm
- net +5V: track 40.1 -> 41.3 mm, vias 16 -> 17
Other:
- board text added: "High"
- board text added: "ROM bank"
- board text added: "low"
