File: ethernet.sch (KiCad schematic (older format))
At the start: 29 parts, among them IC1 SST39SF010A-70-4C-WHE, J7 AVR-JTAG-10, U2 ATF1502ASL-25AU44, U3 ENC624J600-I_PT

Commit message: cleanups, switch for ROM bank
Parts:
- added R4, R5: 10k, Resistor_SMD:R_0402_1005Metric, symbol Device:R
- added S3: SSAJ110100, SW_SSAJ110100, symbol SSAJ110100:SSAJ110100
Connections:
- net +5V: now also R4.2
- net GND: now also R5.2; no longer IC1.10 (A16)
- new net: R4.1, S3.1
- new net: R5.1, S3.2
- new net ROM_BANK: IC1.10 (A16), S3.C
Changed lines of the file:
@@
 	1    0    0    -1
-$EndComp
-$Comp
-L power:GND #PWR0135
-U 1 1 65F13DFD
-P 12125 2400
-F 0 "#PWR0135" H 12125 2150 50  0001 C CNN
-F 1 "GND" H 12130 2227 50  0000 C CNN
-F 2 "" H 12125 2400 50  0001 C CNN
-F 3 "" H 12125 2400 50  0001 C CNN
-	1    12125 2400
-	0    1    1    0
 $EndComp
 Text GLabel 8300 3250 0    50   Input ~ 0
@@
 Text Label 9600 1850 3    50   ~ 0
 TP34
+$Comp
+L SSAJ110100:SSAJ110100 S3
+U 1 1 6633E915
+P 12625 3800
+F 0 "S3" H 12723 3830 50  0000 L CNN
+F 1 "SSAJ110100" H 12723 3739 50  0000 L CNN
+F 2 "SW_SSAJ110100" H 12625 3800 50  0001 L BNN
+F 3 "" H 12625 3800 50  0001 L BNN
+F 4 "0.9 mm" H 12625 3800 50  0001 L BNN "MAXIMUM_PACKAGE_HEIGHT"
+F 5 "ALPS" H 12625 3800 50  0001 L BNN "MANUFACTURER"
+F 6 "N/A" H 12625 3800 50  0001 L BNN "PARTREV"
+F 7 "SSAJ110100" H 12625 3800 50  0001 L BNN "SNAPEDA_PN"
+F 8 "Manufacturer Recommendations" H 12625 3800 50  0001 L BNN "STANDARD"
+F 9 "SSAJ110100" H 12625 3800 50  0001 C CNN "MPN"
+	1    12625 3800
+	1    0    0    -1
+$EndComp
+$Comp
+L Device:R R?
+U 1 1 6633E91C
+P 12375 3700
+AR Path="/5F6B165A/6633E91C" Ref="R?"  Part="1"
+AR Path="/5F679B53/6633E91C" Ref="R?"  Part="1"
+AR Path="/5F69F4EF/6633E91C" Ref="R?"  Part="1"
+AR Path="/60D72F2C/6633E91C" Ref="R?"  Part="1"
+AR Path="/619A5A47/6633E91C" Ref="R?"  Part="1"
+AR Path="/61B604DE/6633E91C" Ref="R?"  Part="1"
+AR Path="/64F8CFB4/6633E91C" Ref="R?"  Part="1"
+AR Path="/6424DB31/6633E91C" Ref="R?"  Part="1"
+AR Path="/64F0AB25/6633E91C" Ref="R?"  Part="1"
+AR Path="/64F0AB25/64B0E5DB/6633E91C" Ref="R?"  Part="1"
+AR Path="/65DC239E/6633E91C" Ref="R4"  Part="1"
+F 0 "R4" V 12455 3700 50  0000 C CNN
+F 1 "10k" V 12375 3700 50  0000 C CNN
+F 2 "Resistor_SMD:R_0402_1005Metric" V 12305 3700 50  0001 C CNN
+F 3 "" H 12375 3700 50  0000 C CNN
+F 4 "0402WGF1002TCE" V 12375 3700 50  0001 C CNN "MPN"
+	1    12375 3700
+	0    1    1    0
+$EndComp
+$Comp
+L Device:R R?
+U 1 1 6633E923
+P 12375 3900
+AR Path="/5F6B165A/6633E923" Ref="R?"  Part="1"
+AR Path="/5F679B53/6633E923" Ref="R?"  Part="1"
+AR Path="/5F69F4EF/6633E923" Ref="R?"  Part="1"
+AR Path="/60D72F2C/6633E923" Ref="R?"  Part="1"
+AR Path="/619A5A47/6633E923" Ref="R?"  Part="1"
+AR Path="/61B604DE/6633E923" Ref="R?"  Part="1"
+AR Path="/64F8CFB4/6633E923" Ref="R?"  Part="1"
+AR Path="/6424DB31/6633E923" Ref="R?"  Part="1"
+AR Path="/64F0AB25/6633E923" Ref="R?"  Part="1"
+AR Path="/64F0AB25/64B0E5DB/6633E923" Ref="R?"  Part="1"
+AR Path="/65DC239E/6633E923" Ref="R5"  Part="1"
+F 0 "R5" V 12455 3900 50  0000 C CNN
+F 1 "10k" V 12375 3900 50  0000 C CNN
+F 2 "Resistor_SMD:R_0402_1005Metric" V 12305 3900 50  0001 C CNN
+F 3 "" H 12375 3900 50  0000 C CNN
+F 4 "0402WGF1002TCE" V 12375 3900 50  0001 C CNN "MPN"
+	1    12375 3900
+	0    1    1    0
+$EndComp
+$Comp
+L power:+5V #PWR0120
+U 1 1 6633E929
+P 12225 3700
+F 0 "#PWR0120" H 12225 3550 50  0001 C CNN
+F 1 "+5V" V 12240 3828 50  0000 L CNN
+F 2 "" H 12225 3700 50  0001 C CNN
+F 3 "" H 12225 3700 50  0001 C CNN
+	1    12225 3700
+	0    -1   -1   0
+$EndComp
+$Comp
+L power:GND #PWR0121
+U 1 1 6633E92F
+P 12225 3900
+F 0 "#PWR0121" H 12225 3650 50  0001 C CNN
+F 1 "GND" V 12230 3772 50  0000 R CNN
+F 2 "" H 12225 3900 50  0001 C CNN
+F 3 "" H 12225 3900 50  0001 C CNN
+	1    12225 3900
+	0    1    1    0
+$EndComp
+Text GLabel 12525 3800 0    50   Input ~ 0
+ROM_BANK
+Text GLabel 12125 2400 0    50   Input ~ 0
+ROM_BANK
 $EndSCHEMATC
